Commit message: Update inertial_macros.xacro

File: description/inertial_macros.xacro (robot description, xacro)
@@ -3,5 +3,5 @@
     <!-- Specify some standard inertial calculations https://en.wikipedia.org/wiki/List_of_moments_of_inertia -->
     <!-- These make use of xacro's mathematical functionality -->
-<!    <xacro:macro name="inertial_sphere" params="mass radius *origin">
+    <xacro:macro name="inertial_sphere" params="mass radius *origin">
         <inertial>
             <xacro:insert_block name="origin"/>
@@ -11,5 +11,5 @@
                     izz="${(2/5) * mass * (radius*radius)}" />
         </inertial>
-    </xacro:macro>  >!
+    </xacro:macro>
     <xacro:macro name="inertial_box" params="mass x y z *origin">
         <inertial>
